Commit message: Trying manipulation with moveit+lidar+camera

File: src/g1pilot/description_files/urdf/g1_29dof.urdf (robot description, URDF)
Before this commit: robot g1_29dof_rev_1_0, 57 links, 56 joints
Links:
- added link lidar_link, mass 0.2; collision cylinder length=0.05 radius=0.04; visual cylinder length=0.05 radius=0.04
Joints:
- added joint head_to_lidar_joint: type fixed, parent head_link, child lidar_link, origin xyz=0.0 0.0 0.10 rpy=0 0 0
